File: pcb/pain27divided3.kicad_pcb (KiCad board)
At the start: 2 copper layers, 223.8 x 100 mm, 87 parts, among them J1 Screw_Terminal_01x08, J2 Screw_Terminal_01x08, J69 Conn_01x02, J73 Conn_01x02, J80085 Conn_01x02, K1 Q, K10 P, K11 A, K12 S, K13 D, K14 F, K15 G, K16 H, K17 J, K18 K, K19 L, K2 W, K20 Z, K21 X, K22 C, K23 V, K24 B, K25 N, K26 M, K27 SPAAAAAAAAAAAAAAAAAAACE, K3 E, K4 R, K5 T, K6 Y, K7 U, K8 I, K9 O

Commit message: added github url to pcb
its ready
Other:
- board text added: "github.com/Stormpegy"
Changed lines of the file:
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@@
   (general
     (thickness 1.6)
-    (drawings 94)
+    (drawings 95)
     (tracks 410)
     (zones 0)
@@
     (pad 1 thru_hole circle (at 1.166726 -1.166726) (size 0.7 0.7) (drill 0.4) (layers *.Cu *.Mask))
   )
+  (gr_text github.com/Stormpegy (at 79 114.75) (layer B.SilkS)
+    (effects (font (size 0.8 0.8) (thickness 0.15)) (justify mirror))
+  )
   (gr_line (start 195.242 88.097) (end 197.623 88.097) (layer Edge.Cuts) (width 0.15))
